File: hardware/telemeter/Telemeter.sch (EAGLE design)
At the start: 8 parts, among them Q1 TIP122, U1 ATMEGA328P_TQFP

Commit message: eagle updates
Connections:
- net SLN_CTRL: now also U1.PD4(XCK/T0)
Changed lines of the file:
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@@
 <label x="27.94" y="147.32" size="1.778" layer="95" rot="MR0" xref="yes"/>
+</segment>
+<segment>
+<pinref part="U1" gate="U1" pin="PD4(XCK/T0)"/>
+<wire x1="157.48" y1="101.6" x2="177.8" y2="101.6" width="0.1524" layer="91"/>
+<label x="177.8" y="101.6" size="1.778" layer="95" xref="yes"/>
 </segment>
 </net>
